File: v3.5/waste_smg_brd_v3.5.kicad_sch (KiCad schematic)
At the start: 24 parts, among them J1 Conn_01x06, U1 74HC595, U2 74HC595, U3 CA56-12CGKWA

Commit message: complete
Parts:
- added J3: Conn_02x07_Top_Bottom, symbol Connector_Generic:Conn_02x07_Top_Bottom
Connections:
- net GND: now also C1.1, U2.13 (~{OE})
- net RCK: no longer U2.12 (RCLK)
- net at U1.1 (QB): now also R2.1
- net at U1.15 (QA): now also R8.1
- net at U1.2 (QC): now also R3.1
- net at U1.3 (QD): now also R4.1
- net at U1.4 (QE): now also R5.1
- net at U1.5 (QF): now also R6.1
- net at U1.6 (QG): now also R7.1
- net at U1.7 (QH): now also R1.1
- net LED1_QE: now reaches R5.2
- net LED1_QE: now also J3.2 (Pin_2)
- net LED1_QF: now reaches R6.2
- net LED1_QF: now also J3.4 (Pin_4)
- net LED1_QA: now reaches R8.2
- net LED1_QA: now also J3.3 (Pin_3)
- net LED1_QB: now reaches R2.2
- net LED1_QB: now also J3.5 (Pin_5)
- net LED1_QD: now reaches R4.2
- net LED1_QD: now also J3.1 (Pin_1)
- net LED1_QH: now reaches R1.2
- net LED1_QH: now also J3.11 (Pin_11)
- net LED2_QD: now reaches U2.3 (QD)
- net LED2_QD: now also J3.10 (Pin_10)
- net LED2_QE: now reaches U2.4 (QE)
- net LED2_QE: now also J3.13 (Pin_13)
- net LED2_QF: now reaches U2.5 (QF)
- net LED2_QF: now also J3.14 (Pin_14)
- net LED2_QG: now reaches U2.6 (QG)
- net LED2_QG: now also J3.6 (Pin_6)
- net LED2_QH: now reaches U2.7 (QH)
- net LED2_QH: now also J3.9 (Pin_9)
- net LED1_QC: now reaches R3.2
- net LED1_QC: now also J3.12 (Pin_12)
- net LED1_QG: now reaches R7.2
- net LED1_QG: now also J3.7 (Pin_7)
- net SER1 renamed SER_NEXT
Other:
- moved on the sheet: C1, U3
